File: demo/demo/ParadaSat.kicad_sch (KiCad schematic)
At the start: 12 parts, among them J1 Conn_02x20_Odd_Even, U1 BME280, U2 MPU-6050

Commit message: sh
Parts:
- added C2: 220pF, symbol Device:C
- added C3, C4: 1uF, symbol Device:C
Connections:
- net +3V3: now also R4.1, U2.13 (VDD), U2.8 (VLOGIC), C3.1, C4.2; no longer R4.2
- net GND: now also U2.1 (CLKIN), U2.11 (FSYNC), U2.18 (GND), U2.9 (AD0), C2.1, C3.2, C4.1
- net SCL: now also U2.23 (SCL)
- net SDA: now also R4.2, U2.24 (SDA); no longer R4.1
- net at U2.20 (CPOUT): now also C2.2
- no-connect marks 0 -> 3
Other:
- note added: "BME280"
- note added: "Debug"
- note added: "MPU6050"
- note added: "Pin connectors"
- note removed: "Jakub Farník"
- title: Paráda Sat -> Sensor Board
- moved on the sheet: C1, J1, U1, U2
