File: sensor_board/sensor_board.kicad_sch (KiCad schematic)
At the start: 20 parts, among them J1 Conn_02x20_Odd_Even, U1 BME280, U2 MPU-6050

Commit message: sensor board
Parts:
- added C6: 10uF, symbol Device:C
- added C7: 1uF, symbol Device:C
- added C8: 100nF, symbol Device:C
- added C9: C_Feedthrough, symbol Device:C_Feedthrough
- added D4: LED, symbol Device:LED
- added J2: Conn_Coaxial, Connector_Coaxial:U.FL_Hirose_U.FL-R-SMT-1_Vertical, symbol Connector:Conn_Coaxial
- added J3: Conn_Coaxial, Connector_Coaxial:SMA_Amphenol_132134-11_Vertical, symbol Connector:Conn_Coaxial
- added L1: 27nH, symbol Device:L
- added R10: 10R, symbol Device:R
- added R11: 10k, symbol Device:R
- added R6: 4.7K, symbol Device:R
- added R7, R8: 510R, symbol Device:R
- added R9: R, symbol Device:R
- added U3: NEO-7M-0, NEO-7M-0:XCVR_NEO-7M-0, symbol NEO-7M-0:NEO-7M-0
- added U4: RFM95W-868S2, symbol RF_Module:RFM95W-868S2
- C1: value 40.1uF -> 0.1uF
Connections:
- net +3V3: now also C6.1, C7.1, C8.1, R11.1, R9.2, U3.22 (V_BCKP), U3.23 (VCC), U4.13 (3.3V)
- net DIO0: now also U4.14 (DIO0)
- net DIO1: now also U4.15 (DIO1)
- net GND: now also C6.2, C7.2, C8.2, C9.2, J2.2 (Ext), J3.2 (Ext), R6.1, U3.10 (GND), U3.12 (GND), U3.13 (GND), U3.24 (GND), U3.7 (VDD_USB), U4.1 (GND), U4.10 (GND), U4.8 (GND)
- net MISO: now also U4.2 (MISO)
- net MOSI: now also U4.3 (MOSI)
- net NSS: now also U4.5 (NSS)
- net RST: now also U4.6 (RESET)
- net SCK: now also U4.4 (SCK)
- net at U2.9 (AD0): now also R6.2
- net RX1 renamed GPS_TX
- net GPS_TX: now also R7.2
- net TX1 renamed GPS_RX
- net GPS_RX: now also R8.2
- new net: J3.1 (In), U4.9 (ANT)
- new net: R11.2, U3.8 (RESET_N)
- new net: C9.1, R10.2
- new net: C9.3, L1.1
- new net: U3.1 (RESERVED), U3.14 (RESERVED), U3.15 (RESERVED), U3.16 (RESERVED), U3.17 (RESERVED)
- new net: R7.1, U3.20 (TXD/SPIMISO)
- new net: R8.1, U3.21 (RXD/SPIMOSI)
- new net: D4.2 (A), R9.1
- new net PPS: D4.1 (K), U3.3 (TIMEPULSE)
- new net RF_IN: J2.1 (In), L1.2, U3.11 (RF_IN)
- new net VCC_RF: R10.1, U3.9 (VCC_RF)
- no-connect marks 3 -> 27
Other:
- note added: "GPS - Neo7m"
- note added: "RFM95"
- moved on the sheet: C1, C2, C3, C4, C5, D1, D2, D3, H1, H2, H3, H4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

Commit message: sensor
Parts:
- C1, C2, C3, C4, C5, C6, C7, C8: footprint (none) -> Capacitor_SMD:C_0805_2012Metric
- C9: footprint (none) -> Filter:Filter_Mini-Circuits_FV1206-7
- D1, D2, D3, D4: footprint (none) -> LED_THT:LED_D8.0mm
- H1, H2, H3, H4: footprint (none) -> MountingHole:MountingHole_3.2mm_M3_DIN965_Pad
- J1: footprint (none) -> Connector_PinSocket_2.54mm:PinSocket_2x20_P2.54mm_Vertical
- L1: footprint (none) -> Inductor_SMD:L_0603_1608Metric
- R1, R2, R3: value R -> 220; footprint (none) -> Resistor_SMD:R_0603_1608Metric
- R10, R11, R4, R5, R6, R7, R8: footprint (none) -> Resistor_SMD:R_0603_1608Metric
- R9: value R -> 220R; footprint (none) -> Resistor_SMD:R_0603_1608Metric
- U4: footprint (none) -> RF_Module:HOPERF_RFM9XW_SMD
Connections:
- net +3V3: now also R5.1; no longer R5.2
- net DIO0: now also J1.23 (Pin_23); no longer J1.33 (Pin_33)
- net DIO1: now also J1.25 (Pin_25); no longer J1.35 (Pin_35)
- net GPS_RX: now also J1.7 (Pin_7); no longer J1.32 (Pin_32)
- net GPS_TX: now also J1.5 (Pin_5); no longer J1.30 (Pin_30)
- net LED_ERROR: now also J1.31 (Pin_31); no longer J1.28 (Pin_28)
- net LED_SUCCESS: now also J1.35 (Pin_35); no longer J1.24 (Pin_24)
- net LED_WARN: now also J1.33 (Pin_33); no longer J1.26 (Pin_26)
- net MISO: now also J1.28 (Pin_28); no longer J1.23 (Pin_23)
- net MOSI: now also J1.30 (Pin_30); no longer J1.25 (Pin_25)
- net NSS: now also J1.34 (Pin_34); no longer J1.29 (Pin_29)
- net RST: now also J1.36 (Pin_36); no longer J1.31 (Pin_31)
- net SCK: now also J1.32 (Pin_32); no longer J1.27 (Pin_27)
- net SCL: now also J1.27 (Pin_27), R4.2; no longer J1.12 (Pin_12), R5.1
- net SDA: now also J1.29 (Pin_29), R5.2; no longer J1.14 (Pin_14), R4.2
Other:
- moved on the sheet: J1, R4, R5

Commit message: sdlkfj
Changed lines of the file:
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@@
 	(text "Pin connectors\n"
 		(exclude_from_sim no)
-		(at 24.13 15.748 0)
+		(at 21.59 15.748 0)
 		(effects
 			(font

Commit message: sensor
Parts:
- added C10, C13, C14: 0.1uF, Capacitor_SMD:C_0805_2012Metric, symbol Device:C
- added C11: 4.7uF, Capacitor_SMD:C_0805_2012Metric, symbol Device:C
- added C12: 0.22uF, Capacitor_SMD:C_0805_2012Metric, symbol Device:C
- added U5: HMC5883L, footprints:LPCC16_HNW, symbol 2026-03-28_11-09-00:HMC5883L
Connections:
- net +3V3: now also C10.2, C13.1, C14.1, U5.13 (VDDIO), U5.2 (VDD), U5.4 (S1); no longer U1.5 (SDO)
- net GND: now also U1.5 (SDO), C10.1, C11.1, C13.2, C14.2, U5.11 (GND), U5.9 (GND)
- net SCL: now also U5.1 (SCL)
- net SDA: now also U5.16 (SDA)
- new net: C11.2, U5.10 (C1)
- new net: C12.2, U5.12 (SETC)
- new net: C12.1, U5.8 (SETP)
- no-connect marks 27 -> 28
Other:
- moved on the sheet: D1, D2, D3, D4, H1, H2, H3, H4, J3, R1, R2, R3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

Commit message: completed sensor
Parts:
- removed C1, C10, C13, C14, C2, C4, C5: 0.1uF, Capacitor_SMD:C_0805_2012Metric, symbol Device:C
- removed C11: 4.7uF, Capacitor_SMD:C_0805_2012Metric, symbol Device:C
- removed C12: 0.22uF, Capacitor_SMD:C_0805_2012Metric, symbol Device:C
- removed C3: 2.2nF, Capacitor_SMD:C_0805_2012Metric, symbol Device:C
- removed C6: 10uF, Capacitor_SMD:C_0805_2012Metric, symbol Device:C
- removed C7: 1uF, Capacitor_SMD:C_0805_2012Metric, symbol Device:C
- removed C8: 100nF, Capacitor_SMD:C_0805_2012Metric, symbol Device:C
- removed H1, H2, H3, H4: MountingHole_Pad, MountingHole:MountingHole_3.2mm_M3_DIN965_Pad, symbol Mechanical:MountingHole_Pad
- removed J2: Conn_Coaxial, Connector_Coaxial:U.FL_Hirose_U.FL-R-SMT-1_Vertical, symbol Connector:Conn_Coaxial
- removed R1, R2, R3: 220, Resistor_SMD:R_0603_1608Metric, symbol Device:R
- removed R10: 10R, Resistor_SMD:R_0603_1608Metric, symbol Device:R
- removed R11: 10k, Resistor_SMD:R_0603_1608Metric, symbol Device:R
- removed R4, R5: 10K, Resistor_SMD:R_0603_1608Metric, symbol Device:R
- removed R6: 4.7K, Resistor_SMD:R_0603_1608Metric, symbol Device:R
- removed R7, R8: 510R, Resistor_SMD:R_0603_1608Metric, symbol Device:R
- removed R9: 220R, Resistor_SMD:R_0603_1608Metric, symbol Device:R
- added C10: 470nF, PCM_JLCPCB:C_0603, symbol PCM_JLCPCB-Capacitors:0603,470nF
- added C11: 220nF, PCM_JLCPCB:C_0603, symbol PCM_JLCPCB-Capacitors:0603,220nF
- added C15, C16, C17, C18, C19, C20, C21: 100nF, PCM_JLCPCB:C_0603, symbol PCM_JLCPCB-Capacitors:0603,100nF
- added C2: 10uF, PCM_JLCPCB:C_0603, symbol PCM_JLCPCB-Capacitors:0603,10uF,(2)
- added C4: 2.2nF, PCM_JLCPCB:C_0603, symbol PCM_JLCPCB-Capacitors:0603,2.2nF
- added J4: U.FL, PCM_JLCPCB:IPEX-SMD_BWIPX-1-001E, symbol PCM_JLCPCB-Extended:RF, Connector, U.FL
- added M1, M2, M3, M4: HOLE, MountingHole:MountingHole_3.2mm_M3_DIN965_Pad, symbol Mechanical:MountingHole_Pad
- added R1: 4.7kΩ, PCM_JLCPCB:R_0603, symbol PCM_JLCPCB-Resistors:0603,4.7kΩ
- added R10, R7, R8: 10kΩ, PCM_JLCPCB:R_0603, symbol PCM_JLCPCB-Resistors:0603,10kΩ
- added R14, R4, R5, R9: 330Ω, PCM_JLCPCB:R_0603, symbol PCM_JLCPCB-Resistors:0603,330Ω
- added R2: 10Ω, PCM_JLCPCB:R_0603, symbol PCM_JLCPCB-Resistors:0603,10Ω
- added R3, R6: 510Ω, PCM_JLCPCB:R_0603, symbol PCM_JLCPCB-Resistors:0603,510Ω
Connections:
- net +3V3: now also C15.2, C16.1, C18.2, C19.1, C2.1, C20.1, C21.2, R10.1, R7.1, R8.1, R9.1
- net GND: now also C10.2, C15.1, C16.2, C17.2, C18.1, C19.2, C2.2, C20.2, C21.1, C4.2, J4.2 (Ext), M1.1, M2.1, M3.1, M4.1, R1.2
- net GPS_RX: now also R3.2
- net GPS_TX: now also R6.2
- net LED_ERROR: now also R14.1
- net LED_SUCCESS: now also R4.1
- net LED_WARN: now also R5.1
- net RF_IN: now also J4.1 (In)
- net SCL: now also R10.2
- net SDA: now also R8.2
- net VCC_RF: now also R2.1
- net at D2.2 (A): now also R5.2
- net at U5.10 (C1): now also C10.1
- net at U5.12 (SETC): now also C11.1
- net at U5.8 (SETP): now also C11.2
- net at U2.10 (REGOUT): now also C17.1
- net at U2.20 (CPOUT): now also C4.1
- net at U2.9 (AD0): now also R1.1
- net at U3.8 (RESET_N): now also R7.2
- net at D3.2 (A): now also R14.2
- net at C9.1: now also R2.2
- net at U3.20 (TXD/SPIMISO): now also R6.1
- net at U3.21 (RXD/SPIMOSI): now also R3.1
- net at D1.2 (A): now also R4.2
- net at D4.2 (A): now also R9.2
