File: main_board/main_board.kicad_sch (KiCad schematic)
At the start: 42 parts, among them J1 Conn_02x20_Odd_Even, J2 AudioJack2_Ground_SwitchT, J3 USB_C_Receptacle_USB2.0_14P, J4 Conn_01x03, J8 Conn_01x02, SW1 SW_SPST, SW3 SW_SPST, U1 RP2040, U2 W25Q128JVS, Y2 ASE-12MHz

Commit message: main board complete
Parts:
- removed C1, C11: 1uF, Capacitor_SMD:C_0402_1005Metric, symbol Device:C
- removed C10, C15, C2, C3, C5, C6, C7, C8, C9: 100nF, Capacitor_SMD:C_0402_1005Metric, symbol Device:C
- removed C12: 1u, Capacitor_SMD:C_0402_1005Metric, symbol Device:C
- removed C13, C14: 100n, Capacitor_SMD:C_0402_1005Metric, symbol Device:C
- removed C4: C, Capacitor_SMD:C_0402_1005Metric, symbol Device:C
- removed R1, R2, R5: 10K, Resistor_SMD:R_0402_1005Metric, symbol Device:R
- removed R10, R3, R4: 1K, Resistor_SMD:R_0402_1005Metric, symbol Device:R
- removed R6, R7: 5.1K, Resistor_SMD:R_0402_1005Metric, symbol Device:R
- removed R8, R9: 27.4R, Resistor_SMD:R_0402_1005Metric, symbol Device:R
- removed U1: RP2040, Package_DFN_QFN:QFN-56-1EP_7x7mm_P0.4mm_EP3.2x3.2mm, symbol MCU_RaspberryPi:RP2040
- added C11, C3, C4: 1uF, PCM_JLCPCB:C_0603, symbol PCM_JLCPCB-Capacitors:0603,1uF
- added C12, C13, C14, C15, C16, C17, C18, C19, C2, C20, C21, C22: 100nF, PCM_JLCPCB:C_0603, symbol PCM_JLCPCB-Capacitors:0603,100nF
- added R1, R5: 27Ω, PCM_JLCPCB:R_0603, symbol PCM_JLCPCB-Resistors:0603,27Ω
- added R11, R12: 5.1kΩ, PCM_JLCPCB:R_0603, symbol PCM_JLCPCB-Resistors:0603,5.1kΩ
- added R2, R3, R4: 10kΩ, PCM_JLCPCB:R_0603, symbol PCM_JLCPCB-Resistors:0603,10kΩ
- added R6, R7: 1kΩ, PCM_JLCPCB:R_0603, symbol PCM_JLCPCB-Resistors:0603,1kΩ
- added U3: RP2040, PCM_JLCPCB:QFN-56-1EP_7x7mm_P0.4mm_EP3.2x3.2mm_ThermalVias, symbol PCM_JLCPCB-Extended:MCU, RP2040
- renumbered H1 to M1, H2 to M2, H3 to M3, H4 to M4
Connections:
- net +1V1: now also C12.1, C13.1, C4.1, U3.23 (DVDD), U3.45 (VREG_VOUT), U3.50 (DVDD)
- net +3V3: now also C11.1, C14.1, C15.1, C17.1, C18.1, C19.1, C20.1, C21.1, C22.1, C3.1, R2.1, R3.1, R4.1, U3.1 (IOVDD), U3.10 (IOVDD), U3.22 (IOVDD), U3.33 (IOVDD), U3.42 (IOVDD), U3.43 (ADC_AVDD), U3.44 (VREG_IN), U3.48 (USB_VDD), U3.49 (IOVDD)
- net +5V: now also C16.1
- net GND: now also C11.2, C12.2, C13.2, C14.2, C15.2, C16.2, C17.2, C18.2, C19.2, C2.1, C20.2, C21.2, C22.2, C3.2, C4.2, R11.2, R12.2, U3.19 (TESTEN), U3.57 (GND)
- net GPIO25: now also R6.1, U3.37 (GPIO25)
- net GPS_RX: now also U3.11 (GPIO8)
- net GPS_TX: now also U3.12 (GPIO9)
- net LED_ERROR: now also U3.15 (GPIO12)
- net LED_SUCCESS: now also U3.16 (GPIO13)
- net LED_WARN: now also U3.14 (GPIO11)
- net QSPI_SCLK: now also U3.52 (QSPI_SCLK)
- net QSPI_SD0: now also U3.53 (QSPI_SD0)
- net QSPI_SD1: now also U3.55 (QSPI_SD1)
- net QSPI_SD2: now also U3.54 (QSPI_SD2)
- net QSPI_SD3: now also U3.51 (QSPI_SD3)
- net QSPLI_SS: now also R3.2, R7.2, U3.56 (QSPI_SS)
- net RUN: now also SW1.2 (B), C2.2, R4.2, U3.26 (RUN)
- net SCL: now also U3.7 (GPIO5)
- net SDA: now also U3.6 (GPIO4)
- net SWCLK: now also U3.24 (SWCLK)
- net SWDIO: now also U3.25 (SWD)
- net USB_D+: now also R1.1
- net USB_D-: now also R5.1
- net XIN: now also U3.20 (XIN)
- net ZERO_RX: now also U3.2 (GPIO0)
- net ZERO_TX: now also U3.3 (GPIO1)
- net at SW3.2 (B): now also R7.1
- net at J3.B5 (CC2): now also R12.1
- net at D1.2 (A): now also R6.2
- net at Y2.1 (EN): now also R2.2
- net at J3.A5 (CC1): now also R11.1
- new net: R5.2, U3.46 (USB_DM)
- new net: R1.2, U3.47 (USB_DP)
Other:
- note removed: "Blízko k RP2040"
- note removed: "C11 pin 44"
- note removed: "C12 pin 45"
