File: power_board/power_board.kicad_sch (KiCad schematic)
At the start: 3 parts, among them J1 Conn_02x20_Odd_Even

Commit message: sdlkfj
Parts:
- added M1, M2, M3, M4: HOLE, MountingHole:MountingHole_3.2mm_M3_DIN965_Pad, symbol Mechanical:MountingHole_Pad
- J1: footprint (none) -> Connector_PinSocket_2.54mm:PinSocket_2x20_P2.54mm_Vertical
- R4, R5: footprint (none) -> Resistor_SMD:R_0603_1608Metric
Connections:
- net RX1 is gone; now on net MOSI: J1.30 (Pin_30)
- net TX1 is gone; now on net SCK: J1.32 (Pin_32)
- net +3V3: now also R5.1; no longer R5.2
- net DIO0: now also J1.23 (Pin_23); no longer J1.33 (Pin_33)
- net DIO1: now also J1.25 (Pin_25); no longer J1.35 (Pin_35)
- net GND: now also M1.1, M2.1, M3.1, M4.1
- net LED_ERROR: now also J1.31 (Pin_31); no longer J1.28 (Pin_28)
- net LED_SUCCESS: now also J1.35 (Pin_35); no longer J1.24 (Pin_24)
- net LED_WARN: now also J1.33 (Pin_33); no longer J1.26 (Pin_26)
- net MISO: now also J1.28 (Pin_28); no longer J1.23 (Pin_23)
- net MOSI: no longer J1.25 (Pin_25)
- net NSS: now also J1.34 (Pin_34); no longer J1.29 (Pin_29)
- net RST: now also J1.36 (Pin_36); no longer J1.31 (Pin_31)
- net SCK: no longer J1.27 (Pin_27)
- net SCL: now also J1.27 (Pin_27), R4.2; no longer J1.12 (Pin_12), R5.1
- net SDA: now also J1.29 (Pin_29), R5.2; no longer J1.14 (Pin_14), R4.2
- net GPS_TX: now reaches J1.5 (Pin_5)
- net GPS_RX: now reaches J1.7 (Pin_7)
- no-connect marks 0 -> 14
Other:
- moved on the sheet: J1, R4, R5

Commit message: vse
Parts:
- removed J1: Conn_02x20_Odd_Even, Connector_PinSocket_2.54mm:PinSocket_2x20_P2.54mm_Vertical, symbol Connector_Generic:Conn_02x20_Odd_Even
- removed R4, R5: 10K, Resistor_SMD:R_0603_1608Metric, symbol Device:R
- added BT1: Battery_Cell, Battery:BatteryHolder_MPD_BH-18650-PC, symbol Device:Battery_Cell
- added C1: 1uF, PCM_JLCPCB:C_0805, symbol PCM_JLCPCB-Capacitors:0805,1uF
- added C10, C2, C9: 4.7uF, PCM_JLCPCB:C_0805, symbol PCM_JLCPCB-Capacitors:0805,4.7uF
- added C11: 100nF, PCM_JLCPCB:C_0805, symbol PCM_JLCPCB-Capacitors:0805,100nF
- added C3: 22uF, PCM_JLCPCB:C_0805, symbol PCM_JLCPCB-Capacitors:0805,22uF
- added C4: 100nF, PCM_JLCPCB:C_1206, symbol PCM_JLCPCB-Capacitors:1206,100nF
- added C5, C6, C7: 10uF, PCM_JLCPCB:C_1206, symbol PCM_JLCPCB-Capacitors:1206,10uF
- added D1: Green, PCM_JLCPCB:D_0805, symbol PCM_JLCPCB-Diodes:LED,0805,Green
- added D2: Red, PCM_JLCPCB:D_0805, symbol PCM_JLCPCB-Diodes:LED,0805,Red
- added F1: Polyfuse, Fuse:Fuse_1812_4532Metric_Pad1.30x3.40mm_HandSolder, symbol Device:Polyfuse
- added J1: Connector, USB-TYPE-C-16P, PCM_JLCPCB:TYPE-C-SMD_HX-TYPE-C-16PIN, symbol PCM_JLCPCB-Extended:Connector, USB-TYPE-C-16P
- added J2: RBF_Switch, Connector_Phoenix_MSTB:PhoenixContact_MSTBA_2,5_2-G_1x02_P5.00mm_Horizontal, symbol Connector_Generic:Conn_01x02
- added J3: Conn_02x20_Odd_Even, Connector_PinSocket_2.54mm:PinSocket_2x20_P2.54mm_Vertical, symbol Connector_Generic:Conn_02x20_Odd_Even
- added L1, L2: 2.2uH,50mA, PCM_JLCPCB:L_0805, symbol PCM_JLCPCB-Inductors:2.2uH,50mA
- added R1: 1MΩ, PCM_JLCPCB:R_0805, symbol PCM_JLCPCB-Resistors:0805,1MΩ
- added R10: 130kΩ, PCM_JLCPCB:R_0603, symbol PCM_JLCPCB-Resistors:0603,130kΩ
- added R11, R12: 5.1kΩ, PCM_JLCPCB:R_0603, symbol PCM_JLCPCB-Resistors:0603,5.1kΩ
- added R13, R14: 1.5kΩ, PCM_JLCPCB:R_0805, symbol PCM_JLCPCB-Resistors:0805,1.5kΩ
- added R15, R16, R17: 1kΩ, PCM_JLCPCB:R_0603, symbol PCM_JLCPCB-Resistors:0603,1kΩ
- added R2: 180kΩ, PCM_JLCPCB:R_0805, symbol PCM_JLCPCB-Resistors:0805,180kΩ
- added R3: 100Ω, PCM_JLCPCB:R_1206, symbol PCM_JLCPCB-Resistors:1206,100Ω
- added R4: 180kΩ, PCM_JLCPCB:R_0603, symbol PCM_JLCPCB-Resistors:0603,180kΩ
- added R5: 3kΩ, PCM_JLCPCB:R_0603, symbol PCM_JLCPCB-Resistors:0603,3kΩ
- added R6: 120Ω, PCM_JLCPCB:R_1206, symbol PCM_JLCPCB-Resistors:1206,120Ω
- added TH2: 10K, Resistor_THT:R_Axial_DIN0204_L3.6mm_D1.6mm_P2.54mm_Vertical, symbol Device:Thermistor_NTC
- added U1: BQ24074RGT, Package_DFN_QFN:VQFN-16-1EP_3x3mm_P0.5mm_EP1.6x1.6mm, symbol Battery_Management:BQ24074RGT
- added U2: TPS61200DRC, Package_SON:Texas_S-PVSON-N10_ThermalVias, symbol Regulator_Switching:TPS61200DRC
- added U3: TPS63001, Package_SON:Texas_DRC0010J_ThermalVias, symbol Regulator_Switching:TPS63001
- M1, M2, M3, M4: value HOLE -> MountingHole_Pad; now left out of the parts list
Connections:
- net +3V3: now also C6.1, C7.1, J3.21 (Pin_21), J3.22 (Pin_22), U3.1 (VOUT), U3.10 (FB)
- net +5V: now also C3.1, J3.19 (Pin_19), J3.20 (Pin_20), U2.10 (FB), U2.2 (VOUT)
- net DIO0: now also J3.23 (Pin_23)
- net DIO1: now also J3.25 (Pin_25)
- net GND: now also BT1.2 (-), C1.2, C10.2, C11.1, C2.2, C3.2, C4.1, C5.2, C6.2, C7.2, C9.2, J1.A12B1 (GND), J1.A6 (D+), J1.A7 (D-), J1.B12A1 (GND), J1.B6 (D+), J1.B7 (D-), J1.S1 (SHIELD), J3.1 (Pin_1), J3.2 (Pin_2), J3.3 (Pin_3), J3.37 (Pin_37), J3.38 (Pin_38), J3.39 (Pin_39), J3.4 (Pin_4), J3.40 (Pin_40), R10.2, R11.2, R12.2, R2.2, R4.2, R6.1, TH2.2, U1.14 (TMR), U1.17 (VSS), U1.4 (~{CE}), U1.6 (EN1), U1.8 (VSS), U2.11 (PAD), U2.4 (PGND), U2.9 (GND), U3.11 (PGND), U3.3 (PGND), U3.9 (GND)
- net GPS_RX: now also J3.7 (Pin_7)
- net GPS_TX: now also J3.5 (Pin_5)
- net LED_ERROR: now also J3.31 (Pin_31)
- net LED_SUCCESS: now also J3.35 (Pin_35)
- net LED_WARN: now also J3.33 (Pin_33)
- net MISO: now also J3.28 (Pin_28)
- net MOSI: now also J3.30 (Pin_30)
- net NSS: now also J3.34 (Pin_34)
- net RST: now also J3.36 (Pin_36)
- net SCK: now also J3.32 (Pin_32)
- net SCL: now also J3.27 (Pin_27)
- net SDA: now also J3.29 (Pin_29)
- new net: L2.1, U3.2 (L2)
- new net: L2.2, U3.4 (L1)
- new net: C2.1, C5.1, J2.1 (Pin_1), L1.1, R1.2, R3.2, U2.5 (VIN), U2.6 (EN), U2.8 (PS), U3.5 (VIN)
- new net: C4.2, R3.1, U3.6 (EN), U3.7 (PS/SYNC), U3.8 (VINA)
- new net: C9.1, F1.1, U1.2 (BAT), U1.3 (BAT)
- new net: C1.1, U2.1 (VAUX)
- new net: L1.2, U2.3 (L)
- new net: R1.1, R2.1, U2.7 (UVLO)
- new net: J1.B5 (CC2), R12.1
- new net: D2.2, R13.1
- new net: R10.1, R17.1
- new net: R15.1, R6.2
- new net: R15.2, R5.1
- new net: R5.2, U1.15 (ITERM)
- new net: R16.1, R4.1
- new net: R16.2, U1.12 (ILIM)
- new net: R17.2, U1.16 (ISET)
- new net: J1.A5 (CC1), R11.1
- new net: BT1.1 (+), F1.2
- new net: D1.2, R14.1
- new net: TH2.1, U1.1 (TS)
- new net EN2: C10.1, J2.2 (Pin_2), R13.2, R14.2, U1.10 (OUT), U1.11 (OUT), U1.5 (EN2)
- new net VBUS: C11.2, J1.A9B4 (VBUS), J1.B9A4 (VBUS), U1.13 (IN)
- new net ~{CHRG}: D2.1, U1.9 (~{CHG})
- new net ~{PGOOD}: D1.1, U1.7 (~{PGOOD})
- no-connect marks 14 -> 16
Other:
- note added: "Mounting holes"
- title: (none) -> ParádaSat - Power Board
